File: Hardware/V1/ESP32-MUSIC-PLAYER-V1.kicad_pcb (KiCad board)
At the start: 2 copper layers, 100 x 65 mm, 70 parts, among them J1 DC-IN, J10 HDR4, J11 EXP1, J2 JST PH4, J3 JST XH4, J4 SHOU-HAN-TF-PUSH, J7 Keystone 900, J8 Keystone 900, J9 Conn_01x02, M1 CN3903 5V/3A Module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

Commit message: Renamed V24 to Vin
Parts:
- C11: value 10µF -> 100µF/16V
- C2: value 100µF -> 100µF/35V
- C3, C4: value 100µF -> 220µF/16V
- D2: value LED -> LED Green
Connections:
- net V24 renamed Vin
